Commit message: Changed the original position

File: urdf/hopejr_arm.urdf.xacro (robot description, xacro)
@@ -72,4 +72,5 @@
         </link>
         <joint name="${prefix}shoulder_yaw" type="revolute"> <parent link="${prefix}shoulder_yaw"/>
+            <parent link="${prefix}shoulder_yaw"/>
             <child link="${prefix}shoulder_roll"/>
             <origin xyz="0 0.05585 0" rpy="${-pi/2} 0 0"/>
@@ -97,4 +98,5 @@
         </link>
         <joint name="${prefix}shoulder_roll" type="revolute"> <parent link="${prefix}shoulder_roll"/>
+            <parent link="${prefix}shoulder_roll"/>
             <child link="${prefix}upper_elbow"/>
             <origin xyz="0 0 0.0884" rpy="0 0 0"/>
@@ -104,5 +106,5 @@
         <link name="${prefix}lower_elbow">
             <visual>
-                <origin xyz="0 0 0" rpy="0 0 0"/>
+                <origin xyz="0 0 0" rpy="0 ${pi/2} 0"/>
                 <geometry>
                     <mesh filename="package://hopejr_arm_description/meshes/visual/lower_elbow.dae" scale="1 1 1"/>
@@ -110,5 +112,5 @@
             </visual>
             <collision>
-                <origin xyz="0 0 0" rpy="0 0 0"/>
+                <origin xyz="0 0 0" rpy="0 ${pi/2} 0"/>
                 <geometry>
                     <mesh filename="package://hopejr_arm_description/meshes/collision/lower_elbow.stl" scale="1 1 1"/>
@@ -126,9 +128,9 @@
             <origin xyz="0.03765 0 0.11311" rpy="0 0 0"/>
             <axis xyz="0 -1 0"/>
-            <limit effort="10" velocity="1.0" lower="-2.53" upper="-0.16" />
+            <limit effort="10" velocity="1.0" lower="-0.96" upper="1.41" />
         </joint>
         <link name="${prefix}forearm">
             <visual>
-                <origin xyz="0 0 0" rpy="0 0 0"/>
+                <origin xyz="0 0 0" rpy="0 ${pi/2} 0"/>
                 <geometry>
                     <mesh filename="package://hopejr_arm_description/meshes/visual/forearm.dae" scale="1 1 1"/>
@@ -136,5 +138,5 @@
             </visual>
             <collision>
-                <origin xyz="0 0 0" rpy="0 0 0"/>
+                <origin xyz="0 0 0" rpy="0 ${pi/2} 0"/>
                 <geometry>
                     <mesh filename="package://hopejr_arm_description/meshes/collision/forearm.stl" scale="1 1 1"/>
@@ -150,6 +152,6 @@
             <parent link="${prefix}lower_elbow"/>
             <child link="${prefix}forearm"/>
-            <origin xyz="0 0 0.06325" rpy="0 0 0"/>
-            <axis xyz="0 0 -1"/>
+            <origin xyz="0.06325 0 0" rpy="0 0 0"/>
+            <axis xyz="-1 0 0"/>
             <limit effort="10" velocity="1.0" lower="${-pi/4}" upper="${pi/18*21}" />
         </joint>
