Commit message: edit urdf

File: urdf/hopejr_arm.urdf (robot description, URDF)
Before this commit: robot hopejr_arm, 7 links, 6 joints
Joints:
- joint elbow_flex: limit lower=-2.53 upper=-0.16 effort=10 velocity=1.0 -> lower=-0.96 upper=1.41 effort=10 velocity=1.0
- joint wrist_roll: axis 0 0 -1 -> -1 0 0; origin xyz=0 0 0.06325 rpy=0 0 0 -> xyz=0.06325 0 0 rpy=0 0 0

File: urdf/hopejr_arm.urdf.xacro (robot description, xacro)
@@ -162,5 +162,5 @@
         parent_link="base_footprint"
         xyz="0 0 0"
-        rpy="0 0 0"
+        rpy="0 ${pi} 0"
     />
 </robot>
